File: Power.sch (KiCad schematic (older format))
At the start: 17 parts

Commit message: Schematic notes
Other:
- note added: "Power"
Changed lines of the file:
@@
 	1    0    0    -1
 $EndComp
+Text Notes 4950 1100 0    157  ~ 0
+Power
 $EndSCHEMATC

Commit message: Inductor choices
Parts:
- L501: value 2.2uH MSS5131-222ML -> 2.2uH CDRH3D23NP-2R2PC
Changed lines of the file:
@@
 P 6000 3400
 F 0 "L501" H 5900 3500 40  0000 C CNN
-F 1 "2.2uH MSS5131-222ML" H 6000 3350 40  0000 C CNN
+F 1 "2.2uH CDRH3D23NP-2R2PC" H 6000 3350 40  0000 C CNN
 F 2 "" H 6000 3400 60  0000 C CNN
 F 3 "" H 6000 3400 60  0000 C CNN

Commit message: Initial footprint association, last few footprints
Parts:
- C501, C502, C503, C504, C505, C506: footprint (none) -> FT:1206
- D501: footprint (none) -> novepad:POWERDI123_DIODE
- L501: footprint (none) -> novepad:CDRH3D23_IND
- L502, L503, R501, R502: footprint (none) -> FT:0603
- REG501: footprint (none) -> FT:SOT23-3
- SJ501: footprint (none) -> FT:SJ_SHORTED
- TP501, TP502: footprint (none) -> novepad:SMD_TEST_POINT
Changed lines of the file:
@@
 LIBS:valves
 LIBS:novepad-cache
-EELAYER 24 0
+EELAYER 25 0
 EELAYER END
 $Descr A4 11693 8268
@@
 F 0 "REG502" H 4650 3150 60  0000 C CNN
 F 1 "LMR10510YSD" H 4250 3650 60  0000 C CNN
-F 2 "" H 4250 3450 60  0000 C CNN
+F 2 "" H 4250 3450 60  0001 C CNN
 F 3 "" H 4250 3450 60  0000 C CNN
 	1    4250 3450
@@
 F 0 "L501" H 5900 3500 40  0000 C CNN
 F 1 "2.2uH CDRH3D23NP-2R2PC" H 6000 3350 40  0000 C CNN
-F 2 "" H 6000 3400 60  0000 C CNN
+F 2 "novepad:CDRH3D23_IND" H 6000 3400 60  0001 C CNN
 F 3 "" H 6000 3400 60  0000 C CNN
 	1    6000 3400
@@
 F 0 "R502" V 6130 2900 40  0000 C CNN
 F 1 "20K 1%" V 6057 2901 40  0000 C CNN
-F 2 "" V 5980 2900 30  0000 C CNN
+F 2 "FT:0603" V 5980 2900 30  0001 C CNN
 F 3 "" H 6050 2900 30  0000 C CNN
 	1    6050 2900
@@
 F 0 "R501" V 5430 2900 40  0000 C CNN
 F 1 "10K 1%" V 5357 2901 40  0000 C CNN
-F 2 "" V 5280 2900 30  0000 C CNN
+F 2 "FT:0603" V 5280 2900 30  0001 C CNN
 F 3 "" H 5350 2900 30  0000 C CNN
 	1    5350 2900
@@
 F 0 "D501" H 5450 3850 40  0000 C CNN
 F 1 "DFLS160-7" H 5450 3650 40  0000 C CNN
-F 2 "" H 5450 3750 60  0000 C CNN
+F 2 "novepad:POWERDI123_DIODE" H 5450 3750 60  0001 C CNN
 F 3 "" H 5450 3750 60  0000 C CNN
 	1    5450 3750
@@
 F 0 "C502" H 6550 3800 40  0000 L CNN
 F 1 "10uF 10V X5R" V 6400 3450 40  0000 L CNN
-F 2 "" H 6588 3550 30  0000 C CNN
+F 2 "FT:1206" H 6588 3550 30  0001 C CNN
 F 3 "" H 6550 3700 60  0000 C CNN
 	1    6550 3700
@@
 F 0 "REG501" H 4150 5400 40  0000 C CNN
 F 1 "NCP1117ST18T3G DNP" H 4150 5350 40  0000 C CNN
-F 2 "" H 4150 5150 60  0000 C CNN
+F 2 "FT:SOT23-3" H 4150 5150 60  0001 C CNN
 F 3 "" H 4150 5150 60  0000 C CNN
 	1    4150 5150
@@
 F 0 "C501" H 2600 3800 40  0000 L CNN
 F 1 "10uF 10V X5R" V 2450 3450 40  0000 L CNN
-F 2 "" H 2638 3550 30  0000 C CNN
+F 2 "FT:1206" H 2638 3550 30  0001 C CNN
 F 3 "" H 2600 3700 60  0000 C CNN
 	1    2600 3700
@@
 F 0 "L502" H 9250 2500 40  0000 C CNN
 F 1 "BLM18KG121" H 9350 2350 40  0000 C CNN
-F 2 "" H 9350 2400 60  0000 C CNN
+F 2 "FT:0603" H 9350 2400 60  0001 C CNN
 F 3 "" H 9350 2400 60  0000 C CNN
 	1    9350 2400
@@
 F 0 "C505" H 9850 2700 40  0000 L CNN
 F 1 "10uF 10V X5R" V 9700 2350 40  0000 L CNN
-F 2 "" H 9888 2450 30  0000 C CNN
+F 2 "FT:1206" H 9888 2450 30  0001 C CNN
 F 3 "" H 9850 2600 60  0000 C CNN
 	1    9850 2600
@@
 F 0 "TP501" H 10130 2550 40  0000 L CNN
 F 1 "CONN_1" H 10050 2605 30  0001 C CNN
-F 2 "" H 10050 2550 60  0000 C CNN
+F 2 "novepad:SMD_TEST_POINT" H 10050 2550 60  0001 C CNN
 F 3 "" H 10050 2550 60  0000 C CNN
 	1    10050 2550
@@
 F 0 "C503" H 8850 2700 40  0000 L CNN
 F 1 "10uF 10V X5R" V 8700 2350 40  0000 L CNN
-F 2 "" H 8888 2450 30  0000 C CNN
+F 2 "FT:1206" H 8888 2450 30  0001 C CNN
 F 3 "" H 8850 2600 60  0000 C CNN
 	1    8850 2600
@@
 F 0 "SJ501" H 7100 3250 70  0000 L BNN
 F 1 "SJ" H 7100 3450 30  0000 L BNN
-F 2 "" H 7200 3400 60  0000 C CNN
+F 2 "FT:SJ_SHORTED" H 7200 3400 60  0001 C CNN
 F 3 "" H 7200 3400 60  0000 C CNN
 	1    7200 3400
@@
 F 0 "L503" H 9250 3550 40  0000 C CNN
 F 1 "BLM18KG121" H 9350 3400 40  0000 C CNN
-F 2 "" H 9350 3450 60  0000 C CNN
+F 2 "FT:0603" H 9350 3450 60  0001 C CNN
 F 3 "" H 9350 3450 60  0000 C CNN
 	1    9350 3450
@@
 F 0 "C506" H 9850 3750 40  0000 L CNN
 F 1 "10uF 10V X5R" V 9700 3400 40  0000 L CNN
-F 2 "" H 9888 3500 30  0000 C CNN
+F 2 "FT:1206" H 9888 3500 30  0001 C CNN
 F 3 "" H 9850 3650 60  0000 C CNN
 	1    9850 3650
@@
 F 0 "TP502" H 10130 3600 40  0000 L CNN
 F 1 "CONN_1" H 10050 3655 30  0001 C CNN
-F 2 "" H 10050 3600 60  0000 C CNN
+F 2 "novepad:SMD_TEST_POINT" H 10050 3600 60  0001 C CNN
 F 3 "" H 10050 3600 60  0000 C CNN
 	1    10050 3600
@@
 F 0 "C504" H 8850 3750 40  0000 L CNN
 F 1 "10uF 10V X5R" V 8700 3400 40  0000 L CNN
-F 2 "" H 8888 3500 30  0000 C CNN
+F 2 "FT:1206" H 8888 3500 30  0001 C CNN
 F 3 "" H 8850 3650 60  0000 C CNN
 	1    8850 3650

Commit message: Paper-checked connector layout
Parts:
- REG501: footprint FT:SOT23-3 -> (none)
Changed lines of the file:
@@
 F 0 "REG501" H 4150 5400 40  0000 C CNN
 F 1 "NCP1117ST18T3G DNP" H 4150 5350 40  0000 C CNN
-F 2 "FT:SOT23-3" H 4150 5150 60  0001 C CNN
+F 2 "" H 4150 5150 60  0001 C CNN
 F 3 "" H 4150 5150 60  0000 C CNN
 	1    4150 5150

Commit message: First attempt at routing the high speed differential traces
Parts:
- REG501: footprint (none) -> FT:SOT223
- REG502: footprint (none) -> novepad:WSON6
Changed lines of the file:
@@
 F 0 "REG502" H 4650 3150 60  0000 C CNN
 F 1 "LMR10510YSD" H 4250 3650 60  0000 C CNN
-F 2 "" H 4250 3450 60  0001 C CNN
+F 2 "novepad:WSON6" H 4250 3450 60  0001 C CNN
 F 3 "" H 4250 3450 60  0000 C CNN
 	1    4250 3450
@@
 F 0 "REG501" H 4150 5400 40  0000 C CNN
 F 1 "NCP1117ST18T3G DNP" H 4150 5350 40  0000 C CNN
-F 2 "" H 4150 5150 60  0001 C CNN
+F 2 "FT:SOT223" H 4150 5150 60  0001 C CNN
 F 3 "" H 4150 5150 60  0000 C CNN
 	1    4150 5150

Commit message: Routed, passes DRC
Connections:
- net BUCK_FB: now reaches R501.1, R502.1, REG502.1 (FB)
- net BUCK_SW: now reaches D501.K, L501.1, REG502.3 (SW)
- net 18V_OUT: now reaches C502.1, L501.2, R502.2, SJ501.1
Changed lines of the file:
@@
 Connection ~ 4350 4000
 $Comp
-L +1.8VA #PWR077
-U 1 1 544E3D1B
-P 10050 3300
-F 0 "#PWR077" H 10050 3440 20  0001 C CNN
-F 1 "+1.8VA" H 10050 3410 30  0000 C CNN
-F 2 "" H 10050 3300 60  0000 C CNN
-F 3 "" H 10050 3300 60  0000 C CNN
-	1    10050 3300
-	1    0    0    -1
-$EndComp
-$Comp
-L GND #PWR078
+L GND #PWR077
 U 1 1 544E6062
 P 2600 4200
-F 0 "#PWR078" H 2600 4200 30  0001 C CNN
+F 0 "#PWR077" H 2600 4200 30  0001 C CNN
 F 1 "GND" H 2600 4130 30  0001 C CNN
 F 2 "" H 2600 4200 60  0000 C CNN
@@
 Text Notes 4950 1100 0    157  ~ 0
 Power
+$Comp
+L +1.8VA #PWR078
+U 1 1 54785B04
+P 10050 3300
+F 0 "#PWR078" H 10050 3440 20  0001 C CNN
+F 1 "+1.8VA" H 10050 3410 30  0000 C CNN
+F 2 "" H 10050 3300 60  0000 C CNN
+F 3 "" H 10050 3300 60  0000 C CNN
+	1    10050 3300
+	1    0    0    -1
+$EndComp
+Text Label 5200 3400 0    60   ~ 0
+BUCK_SW
+Text Label 5200 3250 0    60   ~ 0
+BUCK_FB
+Text Label 6450 3400 0    60   ~ 0
+18V_OUT
 $EndSCHEMATC
